Commit message: included extension in urdf

File: rethink_ee_description/urdf/pneumatic_gripper/rethink_pneumatic_gripper.xacro (robot description, xacro)
@@ -3,5 +3,8 @@
   <xacro:macro name="rethink_pneumatic_gripper" params="side">
     <xacro:property name="tip_length" value="${0.06 + 0.02}" scope="local"/>
-    <!-- Base of end effector -->
+    <xacro:property name="extension_length" value="${0.045}" scope="local"/>
+    <xacro:property name="collision_cylinder_length" value="${extension_length+0.08}" scope="local"/>
+    <xacro:property name="z_pos_tip_joint" value="${extension_length+tip_length}" scope="local"/>
+   <!-- Base of end effector -->
     <link name="${side}_gripper_base">
       <visual>
@@ -14,5 +17,5 @@
         <origin rpy="0 ${pi} ${pi}" xyz="0.0 0.0 0.04"/>
         <geometry>
-          <cylinder length="0.08" radius="0.02"/>
+          <cylinder length="${collision_cylinder_length}" radius="0.02"/>
         </geometry>
         <material name="darkred">
@@ -34,5 +37,5 @@
     <!-- Pneumatic Gripper Tip joint -->
     <joint name="${side}_endpoint" type="fixed">
-      <origin rpy="0 0 0" xyz="0 0 ${tip_length}"/>
+      <origin rpy="0 0 0" xyz="0 0 ${z_pos_tip_joint}"/>
       <parent link="${side}_gripper_base"/>
       <child link="${side}_gripper"/>

Commit message: adjusted length

File: rethink_ee_description/urdf/pneumatic_gripper/rethink_pneumatic_gripper.xacro (robot description, xacro)
@@ -3,5 +3,5 @@
   <xacro:macro name="rethink_pneumatic_gripper" params="side">
     <xacro:property name="tip_length" value="${0.06 + 0.02}" scope="local"/>
-    <xacro:property name="extension_length" value="${0.045}" scope="local"/>
+    <xacro:property name="extension_length" value="${0.055}" scope="local"/>
     <xacro:property name="collision_cylinder_length" value="${extension_length+0.08}" scope="local"/>
     <xacro:property name="z_pos_tip_joint" value="${extension_length+tip_length}" scope="local"/>
